Commit message: Add oak d w camera nodes and urdf

File: src/firo_description/robots/firo.urdf.xacro (robot description, xacro)
@@ -4,7 +4,8 @@
   <xacro:property name="package_path" value="$(find ${package})" />
   <xacro:property name="mechanical" value="${xacro.load_yaml(package_path+'/config/mechanical.yaml')}" />
-  <xacro:include filename="$(find ${package})/urdf/torso.urdf.xacro" />
-  <xacro:include filename="$(find ${package})/urdf/wheel.urdf.xacro" />
-  <xacro:include filename="$(find ${package})/urdf/materials.urdf.xacro" />
+  <xacro:include filename="${package_path}/urdf/materials.urdf.xacro" />
+  <xacro:include filename="${package_path}/urdf/torso.urdf.xacro" />
+  <xacro:include filename="${package_path}/urdf/wheel.urdf.xacro" />
+  <xacro:include filename="${package_path}/urdf/oak-d-w.urdf.xacro" />
   <link name="base_link" />
   <xacro:firo_torso material="silver">
@@ -23,4 +24,5 @@
     <xacro:white/>
   </xacro:firo_wheel>
+  <xacro:oak-d-w prefix="front"/>
   <joint name="base_link_to_torso" type="fixed">
     <parent link="base_link"/>
@@ -56,4 +58,9 @@
     <axis xyz="0 1 0"/>
     <limit effort="7.5" velocity="7.5"/>
+  </joint>
+  <joint name="torso_to_front_camera" type="fixed">
+    <parent link="torso"/>
+    <child link="front_camera_center"/>
+    <origin xyz="0.3001 0 0.12845" rpy="0 0 0"/>
   </joint>
   <transmission name="front_right_wheel_transmission">
