Commit message: Change laser setup

File: src/firo_description/urdf/oak-d-w.urdf.xacro (robot description, xacro)
@@ -22,5 +22,5 @@
       </inertial>
     </link>
-    <link name="${prefix}_rgb_camera_optical_frame"/>
+    <link name="${prefix}_camera_rgb_camera_optical_frame"/>
     <link name="${prefix}_left_camera_frame" />
     <link name="${prefix}_left_camera_optical_frame"/>
@@ -28,8 +28,8 @@
     <link name="${prefix}_right_camera_optical_frame"/>
     <link name="${prefix}_camera_imu_frame"/>
-    <joint name="${prefix}_rgb_camera_optical_joint" type="fixed">
+    <joint name="${prefix}_camera_rgb_camera_optical_joint" type="fixed">
       <origin xyz="${optical_offset_x} 0 0" rpy="-${pi/2} 0.0 -${pi/2}"/>
       <parent link="${prefix}_camera_center"/>
-      <child link="${prefix}_rgb_camera_optical_frame"/>
+      <child link="${prefix}_camera_rgb_camera_optical_frame"/>
     </joint>
     <joint name="${prefix}_left_camera_joint" type="fixed">
